File: eagle/808_lt.brd (EAGLE design)
At the start: 100 x 80.8 mm, 54 parts, among them IC1 TL071P, IC2 TL072P, Q1 2N3904, Q2 2N3906, Q3 2N3904, SW8 MSS42_SW_4PDT

Commit message: tweaked and gcode
Parts:
- moved C82 5.59 mm to (70.6, 15.2)
- moved OUT_NORM 5.59 mm to (83.3, 25.4)
- moved R234 5.59 mm to (70.6, 27.9)
- moved R235 5.59 mm to (75.7, 33.0)
- moved R238 5.59 mm to (75.7, 20.3)
- moved C74 5.59 mm to (27.4, 31.8)
- moved R214 5.59 mm to (27.4, 40.6)
- moved R231 5.59 mm to (27.4, 11.4)
- moved C72 5.59 mm to (11.4, 34.3)
- moved C73 5.59 mm to (34.4, 48.9)
- moved C75 5.59 mm to (35.1, 19.1)
- moved C76 5.59 mm to (55.4, 50.8)
- moved C77 5.59 mm to (41.7, 38.1)
- moved C78 5.59 mm to (50.3, 50.8)
- moved C81 5.59 mm to (63.0, 25.4)
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Routing:
- net N$271: track 26.6 -> 25.5 mm
- net N$267: track 17.6 -> 18.6 mm
- net GND: track 423.2 -> 424.2 mm
- net N$274: track 9.07 -> 8.12 mm
- net +15V: track 102.9 -> 103.7 mm
- net N$260: track 42.6 -> 41.9 mm
- net N$39: track 32.2 -> 31.6 mm
- net TRIG: track 37.2 -> 37.7 mm
Other:
- board size 100 x 80.8 mm -> 100.8 x 80.8 mm

Commit message: corrected 071 power and added resistors to tune pot for value change
Parts:
- added ACCENT, TRIGGER: LSP10, solpad:LSP10
- added R1, R2: 263R, TR808clone:0207/7
- TUNE: value 500R -> 10k
- moved R225 8.48 mm to (61.7, 38.6), turned to 90 degrees
- moved R234 7.03 mm to (75.9, 32.5), turned to 0 degrees
- moved R235 5.39 mm to (71.9, 29.2)
- moved R224 3.64 mm to (64.5, 38.6)
- moved R231 1.27 mm to (27.4, 12.7)
- moved R218 0.51 mm to (14.2, 34.3)
Connections:
- net +15V: now also IC1.7; no longer IC1.4
- net -15V: now also IC1.4; no longer IC1.7
- net GND: now also R2.1
- net LT: now also TRIGGER.MP
- net N$254: now also R1.1
- net N$255: now also R1.2, R2.2
- net TRIG: now also ACCENT.MP
Routing:
- net N$262: track 100.3 -> 43.2 mm
- net GND: track 424.2 -> 405.1 mm
- net +15V: track 103.7 -> 87.1 mm
- net -15V: track 78.4 -> 73.8 mm
- net TRIG: track 37.7 -> 41.4 mm
- net N$109: track 8.89 -> 5.41 mm
- net N$255: track 9.72 -> 13.2 mm
- net LT: track 23.7 -> 26.7 mm
- net N$39: track 31.6 -> 34.6 mm
- net N$254: track 15.1 -> 16.9 mm
- net N$260: track 41.9 -> 40.7 mm
- net N$251: track 83.0 -> 84.0 mm
- net N$267: track 18.6 -> 18.0 mm
